Commit message: feat(bringup): first real-robot SLAM run - lidar, IMU, EKF, slam_toolbox
Everything in HANDOFF §4 up to now was simulation. This is the stack
running on the actual robot: drive board, VLP-16, IMU, EKF and
slam_toolbox all live on the Jetson, with RViz on a laptop over the
network. New slam.launch.py brings the whole lot up at once.

Four things cost real time today and are written up in HANDOFF §10 so
they do not cost it again:

The IMU is not an iAHRS. It is a LORD MicroStrain 3DM-GV7-AHRS, and
every mention of iAHRS in the docs was wrong - corrected throughout.
Its driver is a plain apt install, no clone needed, but the GV7 refuses
to start until filter_pps_source and filter_declination_source are
turned off: it is an AHRS with no GNSS, so the defaults ask the device
for hardware it does not have and the node aborts on Error(3).

The site guest WiFi drops UDP multicast, which kills ROS 2 discovery
outright - ping works, `ros2 topic list` shows two topics forever.
Fast DDS Discovery Server routes around it. Two traps in doing so:
without a SUPER_CLIENT profile the CLI still sees nothing, and none of
it takes effect until `ros2 daemon stop`, because the daemon caches the
old discovery config.

FTDI's default 16ms latency_timer chops BV replies into 1-3 byte
fragments, which reads exactly like a framing bug - and only in the ROS
node, because probe_drive_board.py's 20ms idle gap happens to hide it.
read_frame() now judges frame end by an inter-byte gap rather than by
matching ETX as a value, but the timer still has to be dropped to 1 by
hand after every replug; the udev ATTR does not reliably take.

A short BV reply is often not a protocol fault at all but the E-stop:
the board answers 02 32 03 LRC with no odometry payload. It says so now
instead of reporting a truncated frame.

The IMU is mounted upside down - 611 of 616 samples over 159 degrees of
rotation had its yaw rate opposing the wheel odometry. Whether the flip
is about X or about Y could not be determined: both invert Z identically,
a full start-to-stop drive integrates to exactly zero acceleration by
definition, and differentiating 1mm/30Hz odometry twice is pure noise
(it reported 19 m/s^2). Since planar SLAM only needs the yaw rate, which
both cases correct the same way, the EKF takes rate only and never
absolute heading - the one quantity the ambiguity would flip. The URDF
applies the flip on the real robot only, leaving the sim TF tree alone.

File: src/tetra_dsv_s_description/urdf/tetra_dsv_s_base.xacro (robot description, xacro)
@@ -186,5 +186,29 @@
   </joint>
   <!-- ==================================================================== -->
-  <!-- On-board IMU (iAHRS). Pose from [URDF] base_link_to_imu_link.          -->
+  <!-- On-board IMU. Pose from [URDF] base_link_to_imu_link.                 -->
+  <!--                                                                       -->
+  <!-- The part is a LORD MicroStrain 3DM-GV7-AHRS, not the iAHRS this file  -->
+  <!-- used to name (confirmed 2026-08-13 on the real robot: /dev/ttyACM0    -->
+  <!-- enumerates as Lord_Inertial_Sensor, model 3DMGV7-AHRS, S/N            -->
+  <!-- 6288.171025). See tetra_dsv_s_bringup/config/imu_gv7.yml.             -->
+  <!--                                                                       -->
+  <!-- MOUNTING: on the real robot the unit is installed UPSIDE DOWN. At     -->
+  <!-- rest it reads az = -9.83 m/s^2 (gravity along -Z), and driving the    -->
+  <!-- robot showed its yaw rate opposing the wheel odometry on 611 of 616   -->
+  <!-- samples over 159 deg of rotation - so the Z axis is definitely        -->
+  <!-- inverted. Whether the flip is about X or about Y was NOT determined:  -->
+  <!-- both invert Z identically, and separating them needs a clean          -->
+  <!-- longitudinal-acceleration measurement we did not get (see             -->
+  <!-- scripts/check_imu_mounting.py). It does not matter for planar SLAM -  -->
+  <!-- both give the same yaw-rate correction - so roll(180) is used here    -->
+  <!-- and the EKF is configured to take only the yaw RATE from this sensor  -->
+  <!-- (config/ekf.yaml), never its absolute heading, which is the one       -->
+  <!-- quantity the X/Y ambiguity would flip.                                -->
+  <!--                                                                       -->
+  <!-- Gazebo's IMU is an idealised part mounted the normal way up, so the   -->
+  <!-- flip is applied only when this file is expanded for the real robot.   -->
+  <!-- Keeping it out of the sim leaves the two TF trees the same shape.     -->
+  <xacro:property name="imu_mount_rpy"
+                  value="${'0 0 0' if '$(arg use_gazebo)' == 'true' else '3.14159265 0 0'}"/>
   <!-- ==================================================================== -->
   <link name="imu_link"/>
@@ -192,5 +216,5 @@
     <parent link="base_link"/>
     <child  link="imu_link"/>
-    <origin xyz="0 0 0.232" rpy="0 0 0"/>
+    <origin xyz="0 0 0.232" rpy="${imu_mount_rpy}"/>
   </joint>
 </robot>
